File: pcb slot in/whykb.kicad_pcb (KiCad board)
At the start: 2 copper layers, 89 parts, among them K1 KEYSW, K10 KEYSW, K11 KEYSW, K12 KEYSW, K13 KEYSW, K14 KEYSW, K15 KEYSW, K16 KEYSW, K17 KEYSW, K18 KEYSW, K19 KEYSW, K2 KEYSW, K20 KEYSW, K21 KEYSW, K22 KEYSW, K23 KEYSW, K24 KEYSW, K25 KEYSW, K26 KEYSW, K27 KEYSW, K28 KEYSW, K29 KEYSW, K3 KEYSW, K30 KEYSW, K31 KEYSW, K32 KEYSW, K33 KEYSW, K34 KEYSW, K35 KEYSW, K36 KEYSW, K37 KEYSW, K38 KEYSW, K39 KEYSW, K4 KEYSW, K40 KEYSW, K41 KEYSW, K42 KEYSW, K5 KEYSW, K6 KEYSW, K7 KEYSW, K8 KEYSW, K9 KEYSW, SW1 SW_PUSH, SW2 RotaryEncoder_Switch, U1 sea-picro, U2 SSD1306 128x32

Commit message: routed traces
Parts:
- removed R1: 10k, keebio_parts:R_0805
- removed SW1: SW_PUSH, Button_Switch_SMD:SW_SPST_TL3342
- D1, D10, D11, D12, D13, D14, D15, D16, D17, D18, D19, D2, D20, D21, D22, D23, D24, D25, D26, D27, D28, D29, D3, D30, D31, D32, D33, D34, D35, D36, D37, D38, D39, D4, D40, D41, D42, D5, D6, D7, D8, D9, U1: moved to B.Cu
- moved D36 443.1 mm to (349.2, 181.4), turned to 90 degrees
- moved D37 430.5 mm to (330.2, 181.4), turned to 90 degrees
- moved D13 404.8 mm to (325.4, 138.6), turned to 90 degrees
- moved D24 402.4 mm to (330.2, 162.4), turned to 90 degrees
- moved D39 377.3 mm to (285.8, 176.7), turned to 90 degrees
- moved D33 359.5 mm to (139.7, 157.6), turned to 90 degrees
- moved D40 358.0 mm to (266.7, 176.7), turned to 90 degrees
- moved D38 357.6 mm to (311.1, 181.4), turned to 90 degrees
- moved D3 353.2 mm to (277.8, 119.5), turned to 90 degrees
- moved D21 345.8 mm to (149.2, 138.6), turned to 90 degrees
- moved D25 344.3 mm to (306.4, 157.6), turned to 90 degrees
- moved D28 343.0 mm to (234.9, 157.6), turned to 90 degrees
- moved D14 343.0 mm to (282.6, 138.6), turned to 90 degrees
- moved D26 340.8 mm to (273.1, 157.6), turned to 90 degrees
- moved D1 337.6 mm to (325.4, 119.5), turned to 90 degrees
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Connections:
- SW2 pad C: +5V -> GND
- SW2 pad S2: +5V -> GND
- U1 pad 11: row3 -> row1
- U1 pad 12: col0 -> col1
- U1 pad 13: col1 -> col0
- U1 pad 21: col11 -> col7
- U1 pad 23: col10 -> col8
- U1 pad 25: col8 -> col10
- U1 pad 26: col7 -> col11
- U1 pad 27: unconnected-(U1-Pad27) -> VCC
- U1 pad 29: Net-(R1-Pad2) -> unconnected-(U1-Pad29)
- U1 pad 30: +5V -> GND
- U1 pad 4: +5V -> GND
- U1 pad 5: +5V -> GND
- U1 pad 9: row1 -> row3
- U2 pad 1: SDA -> GND
- U2 pad 2: SCL -> VCC
- U2 pad 3: VCC -> SCL
- U2 pad 4: +5V -> SDA
Routing:
- net row3: track 0.00 -> 302.2 mm
- net col10: track 0.00 -> 301.5 mm
- net col11: track 0.00 -> 300.3 mm
- net col9: track 0.00 -> 291.3 mm
- net row2: track 0.00 -> 285.0 mm
- net row0: track 0.00 -> 283.7 mm
- net col6: track 0.00 -> 272.9 mm
- net col8: track 0.00 -> 252.6 mm
- net row1: track 0.00 -> 249.4 mm
- net col2: track 0.00 -> 246.7 mm
- net col3: track 0.00 -> 245.8 mm
- net col7: track 0.00 -> 236.8 mm
- net col5: track 0.00 -> 233.0 mm
- net col4: track 0.00 -> 217.4 mm
- net col1: track 0.00 -> 193.0 mm
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Other:
- board outline added: 276.9 x 88.9 mm

Commit message: update pcb
cleaned up traces
added some silkscreen
generate gerbers
Parts:
- added G***: LOGO, LOGO, F.Cu at (86.4, 182.6)
- added G***: LOGO, LOGO, F.Cu at (109.3, 189.7)
- added G***: LOGO, LOGO, B.Cu at (266.7, 152.4)
- added G***: LOGO, LOGO, B.Cu at (152.4, 152.4)
- D1, D10, D11, D12, D13, D14, D15, D16, D17, D18, D19, D2, D20, D21, D22, D23, D24, D25, D26, D27, D28, D29, D3, D30, D31, D32, D33, D34, D35, D36, D37, D38, D39, D4, D40, D41, D42, D5, D6, D7, D8, D9: footprint keyboard_parts:D_SOD123_axial -> keyboard_parts:D_SOD123
Routing:
- net row2: track 285.0 -> 301.8 mm
- net row1: track 249.4 -> 264.5 mm
- net row0: track 283.7 -> 298.4 mm
- net row3: track 302.2 -> 309.8 mm
- net Net-(D34-Pad2): track 7.47 -> 9.73 mm
- net Net-(D16-Pad2): track 7.47 -> 9.73 mm
- net Net-(D33-Pad2): track 7.47 -> 9.67 mm
- net Net-(D28-Pad2): track 7.47 -> 9.67 mm
- net Net-(D38-Pad2): track 7.47 -> 9.67 mm
- net Net-(D37-Pad2): track 7.47 -> 9.67 mm
- net Net-(D36-Pad2): track 7.47 -> 9.67 mm
- net Net-(D35-Pad2): track 9.86 -> 12.1 mm
- net Net-(D32-Pad2): track 7.47 -> 9.67 mm
- net Net-(D31-Pad2): track 7.47 -> 9.67 mm
- net Net-(D30-Pad2): track 7.47 -> 9.67 mm
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
Commit message: minor fixes
- updated gerber setting 'subtract soldermask from silkscreen'
- changed silkscreen
Parts:
- turned G*** to 0 degrees
Changed lines of the file:
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@@
       (usegerberattributes true)
       (usegerberadvancedattributes true)
-      (creategerberjobfile true)
+      (creategerberjobfile false)
       (svguseinch false)
       (svgprecision 6)
@@
       (plotinvisibletext false)
       (sketchpadsonfab false)
-      (subtractmaskfromsilk false)
+      (subtractmaskfromsilk true)
       (outputformat 1)
       (mirror false)
@@
   )
   (footprint "LOGO" (layer "B.Cu")
-    (at 152.4 152.4 180)
+    (at 152.4 152.4)
     (attr board_only exclude_from_pos_files exclude_from_bom)
     (fp_text reference "G***" (at 0 0) (layer "B.SilkS") hide
